File: ENYA-SIMR-GTWL-PCRC.kicad_pcb (KiCad board)
At the start: 2 copper layers, 112.4 x 12 mm, 29 parts, among them J1 PICO_BLADE_1x3_MALE_RA_SMD

Commit message: WIP
Parts:
- G1: moved to B.Cu
- G2: footprint ENYA_Bitmap:CC-BY-SA_12MM -> ENYA_Bitmap:CC-BY-SA_6MM; moved to B.Cu
- moved G1 69.9 mm to (220.5, 134.2), turned to 180 degrees
- moved G2 58.7 mm to (232.6, 134.5), turned to 180 degrees
- moved J1 9.58 mm to (179.4, 140.2)
- moved C1 3.56 mm to (180.4, 132.7)
- moved D3 1.64 mm to (194.8, 132.7), turned to -177 degrees
- moved D10 1.58 mm to (253.8, 132.7), turned to 177 degrees
- moved C5 1.56 mm to (211.6, 132.0)
- moved C4 1.56 mm to (203.2, 132.3)
- moved C12 1.56 mm to (270.5, 133.7)
- moved C6 1.56 mm to (220.1, 131.9)
- moved C9 1.56 mm to (245.4, 132.3)
- moved C3 1.56 mm to (194.8, 132.7)
- moved D2 1.54 mm to (186.4, 133.2), turned to -176 degrees
- moved D1 1.50 mm to (178.0, 133.8), turned to -175 degrees
- moved D11 1.50 mm to (262.2, 133.2), turned to 176 degrees
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Connections:
- J1 pad 1: +5V -> GND
- J1 pad 3: GND -> +5V
Routing:
- net +5V: track 133.4 -> 140.0 mm
- net Net-(D10-DOUT): track 10.7 -> 6.19 mm
- net Net-(D10-DIN): track 10.5 -> 6.09 mm
- net Net-(D1-DOUT): track 10.4 -> 6.24 mm
- net Net-(D2-DOUT): track 10.3 -> 6.26 mm
- net Net-(D5-DOUT): track 9.08 -> 6.21 mm
- net Net-(D4-DOUT): track 9.03 -> 6.17 mm
- net Net-(D6-DOUT): track 8.82 -> 6.16 mm
- net Net-(D7-DOUT): track 8.78 -> 6.27 mm
- net Net-(D8-DOUT): track 8.65 -> 6.32 mm
- net /LED_DI: track 8.93 -> 6.98 mm
- net Net-(D11-DOUT): track 5.13 -> 6.17 mm
- net GND: vias 69 -> 56
Other:
- board size 112.4 x 12 mm -> 101.6 x 14.5 mm
- board text added: "ENYA-SIMR- GTWL-PCRC rev.1.0a"
