File: ENYA-SIMR-GTWL-PCRC.kicad_sch (KiCad schematic)
At the start: 29 parts, among them J1 PICO_BLADE_1x3_MALE_RA_SMD

Commit message: WIP
Parts:
- G2: footprint ENYA_Bitmap:CC-BY-SA_12MM -> ENYA_Bitmap:CC-BY-SA_6MM
Connections:
- net +5V: now also J1.3 (Pin_3); no longer J1.1 (Pin_1)
- net GND: now also J1.1 (Pin_1); no longer J1.3 (Pin_3)
Other:
- moved on the sheet: J1
Changed lines of the file:
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@@
       (effects (font (size 1.524 1.524)) hide)
     )
-    (property "Footprint" "ENYA_Bitmap:CC-BY-SA_12MM" (at 391.16 226.06 0)
+    (property "Footprint" "ENYA_Bitmap:CC-BY-SA_6MM" (at 391.16 226.06 0)
       (effects (font (size 1.27 1.27)) hide)
     )
@@
     )
   )
-  (symbol (lib_id "ENYA_Connector_PicoBlade:PICO_BLADE_1x3_MALE_RA_SMD") (at 38.1 129.54 0) (mirror y) (unit 1)
-    (in_bom yes) (on_board yes) (dnp no) (fields_autoplaced)
-    (property "Reference" "J1" (at 38.1 122.15 0)
+  (symbol (lib_id "ENYA_Connector_PicoBlade:PICO_BLADE_1x3_MALE_RA_SMD") (at 38.1 129.54 180) (unit 1)
+    (in_bom yes) (on_board yes) (dnp no)
+    (property "Reference" "J1" (at 38.1 136.93 0)
       (effects (font (size 1.27 1.27)))
     )
-    (property "Value" "PICO_BLADE_1x3_MALE_RA_SMD" (at 38.1 134.62 0)
+    (property "Value" "PICO_BLADE_1x3_MALE_RA_SMD" (at 38.1 124.46 0)
       (effects (font (size 1.27 1.27)) hide)
     )
@@
       (effects (font (size 1.27 1.27)) hide)
     )
-    (property "Manufacturer Part Number" "0532610371" (at 38.1 124.198 0)
+    (property "Manufacturer Part Number" "0532610371" (at 38.1 134.882 0)
       (effects (font (size 1.27 1.27)))
     )
